File: VCARSMD.kicad_pcb (KiCad board)
At the start: 2 copper layers, 146.4 x 128.5 mm, 94 parts, among them J1 Conn_01x10_Pin, J15 Conn_02x05_Odd_Even, J3 Conn_01x10_Pin, J4 AudioJack2, J5 AudioJack2, J6 AudioJack2, J7 AudioJack2, J8 AudioJack2, J9 AudioJack2, Q1 BC857, Q2 BC847, Q3 BC857, Q4 BC847, Q5 BC847, Q6 BC847, SW1 SW_SPDT, SW2 SW_SPDT, U3 4001, U5 TL074, U6 TL074

Commit message: Add files via upload
Parts:
- removed J1, J3: Conn_01x10_Pin, Connector_PinHeader_2.54mm:PinHeader_1x10_P2.54mm_Vertical
- added ?: , , F.Cu at (155.2, 101.7)
- added ?: , , F.Cu at (106.3, 101.7)
- added J101: Conn_01x11_Pin, Connector_PinSocket_2.54mm:PinSocket_1x11_P2.54mm_Vertical, F.Cu at (132.8, 76.2)
- added J102: Conn_01x11_Pin, Connector_PinSocket_2.54mm:PinSocket_1x11_P2.54mm_Vertical, F.Cu at (181.7, 76.2)
- C1, D1, Q2, Q3, R1, R2, R3, R4, R5, R6, U3: moved to F.Cu
- moved R3 60.0 mm to (176.3, 94.2), turned to 0 degrees
- moved R1 59.2 mm to (161.7, 95.1)
- moved Q2 58.9 mm to (157.5, 95.4), turned to -90 degrees
- moved C1 58.5 mm to (176.3, 96.6)
- moved R4 57.1 mm to (181.2, 98.9)
- moved U3 56.8 mm to (168.4, 97.3)
- moved R2 56.6 mm to (161.7, 97.5)
- moved D1 56.2 mm to (176.3, 98.9)
- moved R6 54.2 mm to (161.7, 100.0)
- moved R5 54.2 mm to (176.3, 101.1)
- moved Q3 49.9 mm to (166.2, 104.5), turned to 90 degrees
- moved R26 4.57 mm to (176.3, 91.7)
- moved C2 4.42 mm to (160.9, 90.9)
- moved D5 4.42 mm to (176.3, 79.9)
- moved Q1 4.42 mm to (156.4, 86.1)
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Connections:
- net Net-(SW1-B) renamed SW12
- net Net-(SW2-C) renamed SW32
Routing:
- net SW32: track 16.7 -> 118.5 mm, vias 0 -> 4
- net SW12: track 6.69 -> 106.9 mm, vias 0 -> 4
- net HICOMP: track 78.2 -> 17.2 mm, vias 1 -> 2
- net RCV: track 30.1 -> 38.5 mm
- net GND: track 13.2 -> 20.7 mm, vias 4 -> 6
- net VGNDR: track 104.8 -> 100.5 mm
- net ACV: track 41.2 -> 45.4 mm
- net OUT: track 144.0 -> 147.0 mm, vias 2 -> 3
- net FBO: track 102.6 -> 99.8 mm
- net Net-(D1-K): track 7.39 -> 9.89 mm
- net GOAL: track 88.5 -> 86.3 mm
- net EOC: track 46.0 -> 44.2 mm
- net Net-(R17-Pad2): track 6.52 -> 8.15 mm
- net IN: track 135.7 -> 134.4 mm
- net VGNDA: track 64.3 -> 65.3 mm
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Other:
- board size 146.4 x 128.5 mm -> 143.2 x 128.5 mm
