File: VCARSMD.kicad_sch (KiCad schematic)
At the start: 71 parts, among them J1 Conn_01x10_Pin, J15 Conn_02x05_Odd_Even, J3 Conn_01x10_Pin, J4 AudioJack2, J5 AudioJack2, J6 AudioJack2, J7 AudioJack2, J8 AudioJack2, J9 AudioJack2, Q1 BC857, Q2 BC847, Q3 BC857, Q4 BC847, Q5 BC847, Q6 BC847, SW1 SW_SPDT, SW2 SW_SPDT, U3 4001, U5 TL074, U6 TL074

Commit message: Add files via upload
Parts:
- removed J1, J3: Conn_01x10_Pin, Connector_PinHeader_2.54mm:PinHeader_1x10_P2.54mm_Vertical, symbol Connector:Conn_01x10_Pin
- added J101, J102: Conn_01x11_Pin, Connector_PinSocket_2.54mm:PinSocket_1x11_P2.54mm_Vertical, symbol Connector:Conn_01x11_Pin
Connections:
- net +12V: now also J101.2 (Pin_2), J102.2 (Pin_2)
- net -12V: now also J101.10 (Pin_10), J102.10 (Pin_10)
- net EOC: now also J101.5 (Pin_5), J102.5 (Pin_5)
- net FBO: now also J101.9 (Pin_9), J102.9 (Pin_9)
- net GND: now also J101.11 (Pin_11), J102.11 (Pin_11)
- net GOAL: now also J101.6 (Pin_6), J102.6 (Pin_6)
- net OUT: now also J101.4 (Pin_4), J102.4 (Pin_4)
- net VGNDA: now also J101.8 (Pin_8), J102.8 (Pin_8)
- net VGNDR: now also J101.7 (Pin_7), J102.7 (Pin_7)
- net SW12: now reaches R1.2, SW1.2 (B)
- net SW12: now also J101.3 (Pin_3), J102.3 (Pin_3)
- net SW32: now reaches SW2.3 (C), U3.3, U3.5
- net SW32: now also J101.1 (Pin_1), J102.1 (Pin_1)
